File: ext_module.kicad_pcb (KiCad board)
At the start: 2 copper layers, 112 x 52 mm, 23 parts, among them P1 USB_B, P10 CONN_T_c_leddim, P2 CONN_USB_B, P3 CONN_USB_HUB, P4 CONN_USB_FDRIVE, P5 CONN_TEENSY_DATA, P6 CONN_usb_fdrv, P7 CONN_T_c_fdrv, P8 CONN_teensy, P9 CONN_t_c_eeprom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

Commit message: tweak ext mod
Parts:
- R10k2: moved to F.Cu
- moved P7 36.7 mm to (97.0, 26.0)
- moved Photo_R1 10.1 mm to (71.6, 26.0)
- moved R10k2 8.36 mm to (71.6, 31.3)
- moved R100k1 8.25 mm to (108.5, 36.9), turned to 90 degrees
- moved U2 5.08 mm to (27.2, 28.6), turned to 180 degrees
- moved P5 2.54 mm to (38.6, 42.3), turned to 90 degrees
Routing:
- net GND: track 31.5 -> 48.2 mm, vias 6 -> 7
- net Net-(R100k1-Pad1): track 20.5 -> 11.2 mm
- net Net-(P5-Pad2): track 45.6 -> 39.4 mm
- net Net-(P7-Pad1): track 14.0 -> 20.2 mm
- net Net-(P10-Pad1): track 30.0 -> 25.4 mm
- net Net-(D1-Pad1): track 74.2 -> 76.5 mm
- net Net-(P5-Pad1): track 38.8 -> 39.9 mm, vias 0 -> 2
